Commit message: checking collisions

File: src/robots/a1_description/urdf/a1_1.urdf (robot description, URDF)
Before this commit: robot a1, 6 links, 5 joints
Links:
- removed link FR_calf
- removed link FR_foot
Joints:
- removed joint FR_calf_joint
- removed joint FR_foot_fixed
- joint FR_thigh_joint: origin xyz=0 -0.0838 0 rpy=0 0 0 -> xyz=0 -0.11 0 rpy=0 0 0

Commit message: changing joints

File: src/robots/a1_description/urdf/a1_1.urdf (robot description, URDF)
Before this commit: robot a1, 4 links, 3 joints
Links:
- added link FR_calf, mass 0.166; collision box size=0.2 0.016 0.016; visual mesh filename=package://a1_description/meshes/calf.dae scale=1 1 1
- added link FR_foot, mass 0.06; collision sphere radius=0.02; visual sphere radius=0.01
Joints:
- added joint FR_calf_joint: type revolute, parent FR_thigh, child FR_calf, origin xyz=0 0 -0.2 rpy=0 0 0, axis 0 1 0, limit lower=-2.69653369433 upper=-0.916297857297 effort=33.5 velocity=21
- added joint FR_foot_fixed: type fixed, parent FR_calf, child FR_foot, origin xyz=0 0 -0.2 rpy=0 0 0
- joint FR_thigh_joint: origin xyz=0 -0.11 0 rpy=0 0 0 -> xyz=0 -0.0028 0 rpy=0 0 0; parent FR_hip -> FR_thigh_shoulder

File: src/robots/a1_description/urdf/a1_simple.urdf (robot description, URDF)
Before this commit: robot a1, 22 links, 21 joints
Links:
- removed link imu_link
Joints:
- removed joint imu_joint
