Commit message: better urdf

File: src/robots/a1_description/urdf/a1_simple.urdf (robot description, URDF)
Before this commit: robot a1, 21 links, 20 joints
Joints:
- joint FL_thigh_joint: origin xyz=0 0.0838 0 rpy=0 0 0 -> xyz=0 0.0028 0 rpy=0 0 0; parent FL_hip -> FL_thigh_shoulder
- joint FR_thigh_joint: origin xyz=0 -0.0838 0 rpy=0 0 0 -> xyz=0 -0.0028 0 rpy=0 0 0; parent FR_hip -> FR_thigh_shoulder
- joint RL_thigh_joint: origin xyz=0 0.0838 0 rpy=0 0 0 -> xyz=0 0.0028 0 rpy=0 0 0; parent RL_hip -> RL_thigh_shoulder
- joint RR_thigh_joint: origin xyz=0 -0.0838 0 rpy=0 0 0 -> xyz=0 -0.0028 0 rpy=0 0 0; parent RR_hip -> RR_thigh_shoulder
